File: starter_gamepad.kicad_sch (KiCad schematic)
At the start: 14 parts, among them SW1 SW_Push, SW2 SW_Push, SW3 SW_Push, U1 MAX30102, U2 SSD1306

Commit message: test something it worked!! omg
Other:
- note removed: "add a random text thingy thingy"
- note removed: "nomnomnom"
Changed lines of the file:
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@@
 	(generator_version "10.0")
 	(paper "A4")
-	(text "nomnomnom\n"
-		(exclude_from_sim no)
-		(at 99.314 54.102 0)
-		(effects
-			(font
-				(size 1.27 1.27)
-			)
-		)
-	)
-	(text "add a random text thingy thingy"
-		(exclude_from_sim no)
-		(at 108.712 35.306 0)
-		(effects
-			(font
-				(size 1.27 1.27)
-			)
-		)
-	)
 	(junction
 		(at 62.23 116.84)
